File: grantrak10/video_output.sch (KiCad schematic (older format))
At the start: 0 parts

Commit message: starting to draw the video output circuits
Parts:
- added C? (x2): C, ~, symbol C
- added R? (x3): R, ~, symbol R
- added U? (x2): 74LS161, ~, symbol 74LS161
- added U? (x3): 74LS93, ~, symbol 74LS93
- added U? (x2): 74LS74, ~, symbol 74LS74
- added U? (x4): 7402, ~, symbol 7402
- added U? (x2): 74LS08, ~, symbol 74LS08
- added U? (x2): 74LS10, ~, symbol 74LS10
- added U?: 74LS86, ~, symbol 74LS86
- added U?: 74HC04, ~, symbol 74HC04
- added U? (x2): 74LS107, ~, symbol 74LS107
- added U? (x5): 74LS04, ~, symbol 74LS04
- added X?: CRYSTAL, ~, symbol CRYSTAL
Connections:
- new net: U?.15 (Tc), U?.7 (Cep)
- new net: U?.12 (Cp), U?.15 (Tc)
- new net: U?.12 (D), U?.6
- new net: U?.11, U?.3
- new net: U?.2 (D), U?.8
- new net: R?.1, R?.1, U?.1, X?.1
- new net: C?.1, R?.2, U?.1, U?.2
- new net: C?.2, R?.1, U?.1
- new net: C?.2, R?.2, U?.2
- new net: U?.1, U?.1, U?.2
- new net: C?.1, X?.2
- new net -512H: U?.1, U?.6 (~Q)
- new net -COMP_SYNC: U?.2
- new net -HBLANK: U?.1, U?.3
- new net -HRESET: U?.1 (~MR), U?.1 (~MR), U?.11 (Cp), U?.13 (Cd), U?.2, U?.5 (Q)
- new net -HSYNC: U?.12, U?.4 (IN1)
- new net -VRESET: U?.8 (~Q)
- new net -VSYNC: U?.1, U?.12
- new net 128H: U?.10, U?.11 (Q3)
- new net 128V: U?.11 (Q3), U?.14 (CP0)
- new net 16H: U?.14 (Q0)
- new net 16V: U?.1 (CP1..3), U?.12 (Q0)
- new net 1H: U?.14 (Q0)
- new net 1V: U?.1 (CP1..3), U?.12 (Q0)
- new net 256H: U?.3 (Q), U?.9, U?.9 (Cp)
- new net 256V: U?.1 (CP1..3), U?.12 (Q0)
- new net 2H: U?.1, U?.13 (Q1)
- new net 2V: U?.9 (Q1)
- new net 32H: U?.13 (Q1), U?.2
- new net 32V: U?.9 (Q1)
- new net 4H: U?.12 (Q2)
- new net 4V: U?.8 (Q2)
- new net 512H: U?.5 (Q)
- new net 512V: U?.4, U?.9 (Q1)
- new net 64H: U?.12 (Q2), U?.2
- new net 64V: U?.8 (Q2)
- new net 8H: U?.11 (Q3)
- new net 8V: U?.11, U?.11 (Q3), U?.14 (CP0), U?.5
- new net CLOCK: U?.2, U?.2, U?.2 (Cp), U?.2 (Cp), U?.3 (Cp)
- new net COMP_SYNC: U?.1, U?.6 (OUT)
- new net GND: R?.2, U?.7 (GND), U?.7 (GND), U?.7 (GND), U?.7 (GND), U?.7 (GND), U?.7 (GND), U?.7 (GND), U?.7 (GND), U?.7 (GND), U?.7 (GND), U?.7 (GND), U?.7 (GND), U?.7 (GND), U?.7 (GND), U?.7 (GND), U?.7 (GND), U?.7 (GND), U?.7 (GND), U?.7 (GND), U?.8 (GND), U?.8 (GND)
- new net HBLANK: U?.1, U?.13, U?.2
- new net HRESET: U?.3, U?.6 (~Q)
- new net P: U?.1 (Cd), U?.1 (J), U?.10 (Cd), U?.10 (Cet), U?.10 (Cet), U?.10 (Sd), U?.11 (K), U?.13 (Cd), U?.4 (K), U?.4 (Sd), U?.7 (Cep), U?.8 (J)
- new net VCC: U?.14 (VCC), U?.14 (VCC), U?.14 (VCC), U?.14 (VCC), U?.14 (VCC), U?.14 (VCC), U?.14 (VCC), U?.14 (VCC), U?.14 (VCC), U?.14 (VCC), U?.14 (VCC), U?.14 (VCC), U?.14 (VCC), U?.14 (VCC), U?.14 (VCC), U?.14 (VCC), U?.14 (VCC), U?.14 (VCC), U?.14 (VCC), U?.16 (VCC), U?.16 (VCC), U?.5 (VCC), U?.5 (VCC), U?.5 (VCC)
- new net VRESET: U?.2 (R0(1)), U?.2 (R0(1)), U?.2 (R0(1)), U?.3, U?.3 (R0(2)), U?.3 (R0(2)), U?.3 (R0(2)), U?.9 (Q)
- new net VSYNC: U?.13, U?.2, U?.5 (IN2)
- no-connect marks 0 -> 13
Other:
- note added: "450"
- note added: "520"
