File: grantrak10/sound_effects.sch (KiCad schematic (older format))
At the start: 4 parts

Commit message: wip
Parts:
- added C? (x5): C, ~, symbol C
- added C?: CP1, ~, symbol CP1
- added D? (x2): DIODE, ~, symbol DIODE
- added R? (x14): R, ~, symbol R
- added RV?: POT, ~, symbol POT
- added U? (x3): RC4136D, symbol RC4136D
Connections:
- net -5V: now also U?.6 (V-), U?.6 (V-), U?.6 (V-)
- net GND: now also C?.1, C?.1, C?.2, R?.1, R?.1, R?.1, R?.1, R?.1
- net at Q?.3 (E): now also R?.2, C?.1
- net VCC: now reaches R?.1
- net VCC: now also U?.11 (V+), U?.11 (V+), U?.11 (V+)
- new net: R?.2, RV?.1, RV?.2, U?.1 (-)
- new net: C?.2, R?.2, U?.2 (+)
- new net: C?.1, C?.1, RV?.3, U?.3
- new net: C?.2, R?.1 (x2)
- new net: C?.2, R?.1, R?.2
- new net: D?.2 (K), R?.1, R?.2, R?.2, U?.1 (-)
- new net: R?.1, R?.2, R?.2, U?.2 (+)
- new net: C?.2, D?.2 (K), R?.1, U?.1 (-)
- new net: R?.1, R?.2, R?.2, U?.3
- new net: C?.1, R?.2, R?.2
- new net: R?.1, R?.1, U?.3
- new net: R?.2, U?.2 (+)
- new net CRASH_A: D?.1 (A)
- new net SCREECH: D?.1 (A)
- new net TO_72046_PIN_13: R?.2, R?.2
Other:
- moved on the sheet: C?, Q?, R?
