File: grantrak10/grantrak10.sch (KiCad schematic (older format))
At the start: 0 parts

Commit message: wip
Changed lines of the file:
@@
 LIBS:contrib
 LIBS:valves
+LIBS:rc4136d
 LIBS:grantrak10-cache
 EELAYER 27 0
@@
 $Descr A4 11693 8268
 encoding utf-8
-Sheet 1 3
+Sheet 1 4
 Title ""
-Date "13 aug 2016"
+Date "14 aug 2016"
 Rev ""
 Comp ""
@@
 F1 "sound_effects.sch" 50
 $EndSheet
+$Sheet
+S 2300 3600 2450 500
+U 57B0DF30
+F0 "Game Logic" 50
+F1 "game_logic.sch" 50
+$EndSheet
 $EndSCHEMATC

Commit message: throwing everything in a single sheet just like the original schamatics from Atari
Parts:
- added C? (x7): C, ~, symbol C
- added C? (x2): CP1, ~, symbol CP1
- added D? (x2): DIODE, ~, symbol DIODE
- added Q?: 2N3643, ?, symbol BC413B
- added R? (x19): R, ~, symbol R
- added RV?: POT, ~, symbol POT
- added U? (x5): 74LS04, ~, symbol 74LS04
- added U? (x2): 74LS107, ~, symbol 74LS107
- added U?: 74HC04, ~, symbol 74HC04
- added U?: 74LS86, ~, symbol 74LS86
- added U? (x2): 74LS10, ~, symbol 74LS10
- added U? (x4): 7402, ~, symbol 7402
- added U? (x2): 74LS74, ~, symbol 74LS74
- added U? (x2): 74LS08, ~, symbol 74LS08
- added U? (x3): 74LS93, ~, symbol 74LS93
- added U? (x2): 74LS161, ~, symbol 74LS161
- added U? (x3): RC4136D, symbol RC4136D
- added X?: CRYSTAL, ~, symbol CRYSTAL
Connections:
- net labels added: -512H, -5V, -COMP_SYNC, -HBLANK, -HRESET, -HSYNC, -VRESET, -VSYNC, 128H, 128V, 16H, 16V, 1H, 1V, 256H, 256V, 2H, 2V, 32H, 32V, 4H, 4V, 512H, 512V, 64H, 64V, 8H, 8V, CLOCK, COMP_SYNC, CRASH_A, GND, HBLANK, HRESET, P, SCREECH, TO_72046_PIN_13, VCC, VRESET, VSYNC
- wire segments 0 -> 277
- no-connect marks 0 -> 13
Other:
- note added: "450"
- note added: "520"

Commit message: schematics transcription sprint at Garoa Hacker Clube :-)
Parts:
- added A2: 74HC00, ~, symbol 74HC00
- added A4, B1, B2, C1, D1: 74LS74, ~, symbol 74LS74
- added A6: 74LS08, ~, symbol 74LS08
- added C2, E1, U? (x2): 74HC04, ~, symbol 74HC04
- added C6: 7402, ~, symbol 7402
- added C9: 330pF, ~, symbol C
- added JP1: JUMPER, ~, symbol JUMPER
- added L1: 74LS107, ~, symbol 74LS107
- added R1, R2: 330R, ~, symbol R
- C47: renamed from C?; value C -> 100pF
- R81, R82: renamed from R?; value R -> 330R
- R83: renamed from R?; value R -> 680R
- X1: renamed from X?; value CRYSTAL -> 14.318MHz
- gave numbers to parts that had none: 9
Connections:
- net labels added: -16H, -1_STOP, -ATRC, -CAR_1_VIDEO, -CRASH_SEQUENCE, -H_SYNC, -LD1B, -RESET_1, -SKID, -SLICK, -START, -VLD1, -V_RESET, 1024V, CAR_1_VIDEO, H_COUNT, LD1B, RESET_1, SPEED_PULSE_FROM_ANALOG, VLD1
- wire segments 277 -> 357
- no-connect marks 13 -> 20
Other:
- note added: "9316"
- note added: "A2-2"
- note added: "A3-2"
- note added: "B3-1"
- note added: "B4-1"
- note added: "C2-1"
- note added: "C3-2"
- note added: "D3-2"
- note added: "D4-2"
- note added: "REMOVE JUMPER TO\nDISABLE SLICK"
- moved on the sheet: C47, C?, D?, F1A, F3, H2, I2, K1A, K2, L2, Q?, R81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

Commit message: updating the schematics (work in progress)
Parts:
- added C1: 500 20V, ~, symbol C
- added C10: .1, ~, symbol C
- added C3, C8: .1uF, ~, symbol C
- added C44: 10uF, ~, symbol CP1
- added C51: 10uF, ~, symbol C
- added C7: 1MF 20V, ~, symbol C
- added CR11, CR12: 1N914, ~, symbol DIODE
- added L8: LM380N, symbol LM380N
- added Q5: 2N3644, TO_SOT_Packages_THT:TO-92_Molded_Narrow, symbol 2N3906
- added R16: 47k, symbol R
- added R3: 2.7, symbol R
- added R4: 50k, ~, symbol POT
- added R52, R63: 1k, ~, symbol R
- added R53: 10k, ~, symbol R
- added R64, R66, R73, R74: 330R, ~, symbol R
- added R65: 4.7k, ~, symbol R
- C11: renamed from C?; value CP1 -> 10uF
- C12, C26: renamed from C?; value C -> .1 MYL
- C14, C46: renamed from C?; value C -> .1F
- C24: renamed from C?; value C -> .005 MYL
- C25: renamed from C?; value C -> .1uF MYL
- C?: value CP1 -> .1
- CR10, CR9: renamed from D?; value DIODE -> 1N914
- F9: renamed from U?; value RC4136D -> LM741
- R17, R29, R38: renamed from R?; value R -> 10k
- R18: renamed from R?; value R -> 470k
- R28: renamed from R?; value R -> 1k
- R34: renamed from R?; value R -> 68k
- R35: renamed from RV?; value POT -> 250k
- R36, R37, R39, R40, R41: renamed from R?; value R -> 47k
- R42: renamed from R?; value R -> 47k 5%
- R43: renamed from R?; value R -> 1M 5%
- R44: renamed from R?; value R -> 560k 5%
- R? (x2): value R -> 1M
- gave numbers to parts that had none: 7
- renumbered I2 to J2
Connections:
- net labels added: +18V, 72046_PIN12, 72046_PIN13, 72046_PIN14, AUDIO_OUT, FINISH_LINE, RT, VIDEO_OUT
- net labels removed: TO_72046_PIN_13
- wire segments 357 -> 495
- no-connect marks 20 -> 23
Other:
- note added: "(*)"
- note added: "(?)"
- note added: "(???)"
- note added: "(WRONG POWER PINS)\n(TODO: FIX THIS SYMBOL!)"
- note added: "(pin 11)"
- note added: "* DELETE TO DISABLE SLICK"
- note added: "+"
- note added: "A2-1"
- note added: "B4-2"
- note added: "D2-2"
- note added: "E1-1"
- note added: "E4-2"
- note added: "I2 or J2 (?)"
- note added: "MYL"
- moved on the sheet: C11, C12, C14, C24, C25, C26, C47, C9, C?, CR10, CR9, F9A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

Commit message: update schematics and add a csound script to simulate the motorengine sounds
Parts:
- added unit 1 of A6
- added unit 4 of A6
- added A7, B7: 74LS74, ~, symbol 74LS74
- added unit 1 of A8
- added B6: 74LS04, ~, symbol 74LS04
- added C41, C45: .1, ~, symbol C
- added unit 4 of C6
- added unit 2 of C7
- added CR13, CR14, CR15: 1N914, ~, symbol DIODE
- added Q6: 2N3644, TO_SOT_Packages_THT:TO-92_Molded_Narrow, symbol 2N3906
- added Q7, Q8: 2N3643, ?, symbol BC413B
- added R59, R67, R68: 220R, ~, symbol R
- added R75: 330R, ~, symbol R
- added R76, R77: 100R, ~, symbol R
- added R?: 1k, ~, symbol R
- added S1B, S3, S?: SW_Push_SPDT, symbol SW_Push_SPDT
Connections:
- net labels added: -COIN, ANT, ATRC, END_GAME, LED, Q, START, pin_L, pin_M
- wire segments 495 -> 644
- no-connect marks 23 -> 26
Other:
- note added: "(pin 10)"
- note added: "(pin K)"
- note added: "(pin N)"
- note added: "1 PLAY"
- note added: "2 PLAY"
- note added: "AUDIO CIRCUITRY"
- note added: "C4-2"
- note added: "COIN-INPUT & GAME/ATTRACT-MODE SIGNALS"
- note added: "RASTER VIDEO SIGNALS"
- note added: "SYSTEM CLOCK GENERATOR"
- note added: "TEST"
- moved on the sheet: A2B, A2D, A4A, A6B, A8B, A8C, A8D, A8E, A8F, B1A, B1B, B2A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
