File: grantrak10/grantrak10.sch (KiCad schematic (older format))
At the start: 105 parts, among them J1 74LS10, J2 74LS93, K1 74LS107, K2 74LS161, Q1 2N3643, Q5 2N3644, Q6 2N3644, Q7 2N3643, Q8 2N3643, X1 14.318MHz

Commit message: wip - drawing schematics while trying to understand the circuits ;-)
Parts:
- added unit 2 of A4
- added CR17, CR18: LED, symbol device:LED
- added J8: 7413, symbol Logic_TTL_IEEE:7413
- added K8: 74LS74, symbol Logic_74xx:74LS74
- added R20, R21: 150R, symbol device:R
Connections:
- net labels added: -CRASH_A, CLOCKWISE, Pin_12, Pin_13, RATE
- wire segments 644 -> 676
- no-connect marks 26 -> 27
Other:
- moved on the sheet: C44, R63, R64, R65, R66, R73, R74
